File: hardware/eagle/front_panel.sch (EAGLE design)
At the start: 22 parts, among them IC1 74HCT595N, IC2 74HCT595N

Commit message: Reorganized project structure.
Parts:
- U$2: device dreimalb:LED_RING_16 -> dreimalbe:LED_RING_16
Changed lines of the file:
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@@
 <part name="SV2" library="con-lstb" deviceset="MA10-2" device=""/>
 <part name="R17" library="resistor" deviceset="R-EU_" device="0207/7" value="100"/>
-<part name="U$2" library="dreimalb" deviceset="LED_RING_16" device=""/>
+<part name="U$2" library="dreimalbe" deviceset="LED_RING_16" device=""/>
 <part name="U$3" library="tsop-1" deviceset="TSOP1738" device=""/>
 </parts>
