File: hardware/eagle/remoteVolume.brd (EAGLE design)
At the start: 100 x 80 mm, 66 parts, among them CN1 NRJ4HF, IC1 MEGA8-P, IC2 L293D, IC3 7805, IC4 OPA2132P, IC5 PGA2311P, IC7 7905, K1 FTR-B4C, K2 FTR-B4C, Q1 20MHz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

Commit message: Reorganized project structure.
Parts:
- JP4: device dreimalb:AVR-ISP-10 -> dreimalbe:AVR-ISP-10
- SV2: device dreimalb:FE10-2W -> dreimalbe:FE10-2W
- U$1: device dreimalb:RK16816MG -> dreimalbe:RK16816MG
- X_OUT: device dreimalb:RCA-2 -> dreimalbe:RCA-2
Other:
- board text added: "@dreimalbe 2014"
- board text removed: "dreimalb 2014"
Changed lines of the file:
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@@
 <rectangle x1="61.595" y1="60.325" x2="64.4525" y2="61.2775" layer="42"/>
 <text x="96.2025" y="8.89" size="1.778" layer="1" font="vector" ratio="14" rot="R90">RemoteVolume</text>
-<text x="99.06" y="8.89" size="1.778" layer="1" font="vector" ratio="14" rot="R90">dreimalb 2014</text>
+<text x="99.06" y="8.89" size="1.778" layer="1" font="vector" ratio="14" rot="R90">@dreimalbe 2014</text>
 </plain>
 <attributes>
@@
 <element name="C8" library="rcl" package="E2,5-6" value="47u" x="24.765" y="9.525" rot="R90"/>
 <element name="X_IN" library="con-conrad" package="RCA-4-117-01" value="RCA-4-117-01" x="77.1525" y="70.1675"/>
-<element name="JP4" library="dreimalb" package="AVR-ISP-10" value="AVR-ISP-10" x="11.43" y="10.4775" rot="R180"/>
-<element name="U$1" library="dreimalb" package="RK16816MG" value="RK16816MG" x="80.9625" y="8.255"/>
+<element name="JP4" library="dreimalbe" package="AVR-ISP-10" value="AVR-ISP-10" x="11.43" y="10.4775" rot="R180"/>
+<element name="U$1" library="dreimalbe" package="RK16816MG" value="RK16816MG" x="80.9625" y="8.255"/>
 <element name="IC1" library="atmel" package="DIL28-3" value="MEGA8-P" x="22.86" y="20.6375" rot="R180">
 <attribute name="OC_NEWARK" value="unknown" x="22.86" y="20.6375" size="1.778" layer="27" rot="R180" display="off"/>
@@
 <attribute name="OC_FARNELL" value="unknown" x="22.86" y="20.6375" size="1.778" layer="27" rot="R180" display="off"/>
 </element>
-<element name="X_OUT" library="dreimalb" package="RCA-2" value="RCA-2" x="50.4825" y="70.1675"/>
+<element name="X_OUT" library="dreimalbe" package="RCA-2" value="RCA-2" x="50.4825" y="70.1675"/>
 <element name="T3" library="transistor" package="TO92" value="BC337" x="36.83" y="29.21" rot="R90"/>
 <element name="R4" library="rcl" package="0207/7" value="2k" x="31.75" y="30.7975" rot="R270"/>
 <element name="C9" library="rcl" package="C025-025X050" value="100n" x="24.4475" y="13.6525"/>
 <element name="C10" library="rcl" package="C025-025X050" value="100n" x="26.67" y="28.8925" rot="R90"/>
-<element name="SV2" library="dreimalb" package="FE10-2W" value="" x="40" y="10.37">
+<element name="SV2" library="dreimalbe" package="FE10-2W" value="" x="40" y="10.37">
 <attribute name="OC_NEWARK" value="unknown" x="40" y="10.37" size="1.778" layer="27" display="off"/>
 <attribute name="MPN" value="" x="40" y="10.37" size="1.778" layer="27" display="off"/>
