File: hardware/eagle/remoteVolume.sch (EAGLE design)
At the start: 66 parts, among them CN1 NRJ4HF, IC1 MEGA8-P, IC2 L293D, IC3 7805, IC4 OPA2132P, IC5 PGA2311P, IC7 7905, K1 FTR-B4C, K2 FTR-B4C, Q1 20MHz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

Commit message: Reorganized project structure.
Parts:
- JP4: device dreimalb:AVR-ISP-10 -> dreimalbe:AVR-ISP-10
- SV2: device dreimalb:FE10-2W -> dreimalbe:FE10-2W
- U$1: device dreimalb:RK16816MG -> dreimalbe:RK16816MG
- X_OUT: device dreimalb:RCA-2 -> dreimalbe:RCA-2
Changed lines of the file:
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@@
 <part name="C8" library="rcl" deviceset="CPOL-EU" device="E2.5-6" value="47u"/>
 <part name="X_IN" library="con-conrad" deviceset="RCA-4-117-01" device=""/>
-<part name="JP4" library="dreimalb" deviceset="AVR-ISP-10" device=""/>
-<part name="U$1" library="dreimalb" deviceset="RK16816MG" device=""/>
+<part name="JP4" library="dreimalbe" deviceset="AVR-ISP-10" device=""/>
+<part name="U$1" library="dreimalbe" deviceset="RK16816MG" device=""/>
 <part name="IC1" library="atmel" deviceset="MEGA8-P" device=""/>
 <part name="GND10" library="supply1" deviceset="GND" device=""/>
 <part name="P+8" library="supply1" deviceset="VCC" device=""/>
-<part name="X_OUT" library="dreimalb" deviceset="RCA-2" device=""/>
+<part name="X_OUT" library="dreimalbe" deviceset="RCA-2" device=""/>
 <part name="T3" library="transistor" deviceset="BC337" device=""/>
 <part name="R4" library="rcl" deviceset="R-EU_" device="0207/7" value="2k"/>
@@
 <part name="P+9" library="supply1" deviceset="VCC" device=""/>
 <part name="C10" library="rcl" deviceset="C-EU" device="025-025X050" value="100n"/>
-<part name="SV2" library="dreimalb" deviceset="FE10-2W" device=""/>
+<part name="SV2" library="dreimalbe" deviceset="FE10-2W" device=""/>
 <part name="IC4" library="burr-brown" deviceset="OPA2132" device="P"/>
 <part name="R9" library="rcl" deviceset="R-EU_" device="0207/7" value="2k"/>
